File: uMule_board/sheets/rs485.kicad_sch (KiCad schematic)
At the start: 5 parts, among them J2 Dynamixel, U23 SP3485CN

Commit message: Finished schematics. Now ready for PCB
Parts:
- removed C46: 100n, Capacitor_SMD:C_0603_1608Metric, symbol Device:C
- removed D7: SM712_SOT23, Package_TO_SOT_SMD:SOT-23, symbol Diode:SM712_SOT23
- removed J2: Dynamixel, Connector_JST:JST_XH_B4B-XH-A_1x04_P2.50mm_Vertical, symbol Connector_Generic:Conn_01x04
- removed R63: 120R, Resistor_SMD:R_0603_1608Metric, symbol Device:R
- removed U23: SP3485CN, Package_SO:SOIC-8_3.9x4.9mm_P1.27mm, symbol Interface_UART:SP3485CN
