File: uMule_board/sheets/outputs.kicad_sch (KiCad schematic)
At the start: 0 parts

Commit message: Started working on PCB. Ditched high power outputs. Focusing on photodiodes. One commit closer to order
Other:
- title: (none) -> uMule_board
Changed lines of the file:
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@@
 	(generator_version "9.0")
 	(paper "A4")
+	(title_block
+		(title "uMule_board")
+		(date "2025-12-14")
+		(rev "1.0")
+		(comment 1 "Original author: Oliwier Woźniak")
+	)
 	(wire
 		(pts
