File: uMule_board/sheets/mcu.kicad_sch (KiCad schematic)
At the start: 33 parts, among them SW1 DBG_BUTT, SW2 RST, U17 STM32G474RETx, U7 FM24C64B, Y1 8MHz

Commit message: All elements connected. Now making more vias and corrections
Connections:
- net PC6/I2C4_SCL: now also U7.6 (SCL)
- net PC7/I2C4_SDA: now also U7.5 (SDA)
- net PC8/I2C3_SCL: no longer U7.6 (SCL)
- net PC9/I2C3_SDA: no longer U7.5 (SDA)
- net PC12/GPIO: now reaches U17.54 (PC12)
- net PB12/RS485_FC renamed PB12/ADC41_IN3_11
- net PB2/GPIO renamed PB2/RS485FC
- net PC3/ADC12_IN9 renamed PC3/GPIO
Changed lines of the file:
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@@
 	)
 	(rectangle
+		(start 201.93 91.44)
+		(end 227.33 93.98)
+		(stroke
+			(width 0)
+			(type dash)
+		)
+		(fill
+			(type none)
+		)
+	)
+	(rectangle
 		(start 201.93 48.26)
 		(end 229.87 53.34)
@@
 	)
 	(rectangle
-		(start 166.37 81.28)
-		(end 139.7 86.36)
+		(start 139.7 81.28)
+		(end 166.37 86.36)
 		(stroke
 			(width 0)
@@
 	)
 	(rectangle
-		(start 201.93 111.506)
-		(end 227.33 119.126)
+		(start 201.93 111.76)
+		(end 227.33 116.586)
 		(stroke
 			(width 0)
@@
 		)
 	)
+	(text "RS485\n"
+		(exclude_from_sim no)
+		(at 227.33 92.964 0)
+		(effects
+			(font
+				(size 1.27 1.27)
+			)
+			(justify right)
+		)
+	)
 	(text "ADC2_IN11/USART1_RX"
 		(exclude_from_sim no)
@@
 	(text "RS485\n"
 		(exclude_from_sim no)
-		(at 227.33 113.03 0)
+		(at 227.33 113.284 0)
 		(effects
 			(font
@@
 	(wire
 		(pts
-			(xy 223.52 97.79) (xy 201.93 97.79)
-		)
-		(stroke
-			(width 0)
-			(type default)
-		)
-	)
-	(wire
-		(pts
 			(xy 88.9 158.75) (xy 88.9 157.48)
 		)
@@
 	(wire
 		(pts
+			(xy 201.93 95.25) (xy 238.76 95.25)
+		)
+		(stroke
+			(width 0)
+			(type default)
+		)
+	)
+	(wire
+		(pts
 			(xy 88.9 168.91) (xy 88.9 167.64)
 		)
@@
 	(wire
 		(pts
+			(xy 201.93 97.79) (xy 238.76 97.79)
+		)
+		(stroke
+			(width 0)
+			(type default)
+		)
+	)
+	(wire
+		(pts
 			(xy 189.23 20.32) (xy 195.58 20.32)
 		)
@@
 	(wire
 		(pts
-			(xy 149.86 20.32) (xy 157.48 20.32)
+			(xy 201.93 100.33) (xy 238.76 100.33)
 		)
 		(stroke
@@
 	(wire
 		(pts
-			(xy 181.61 34.29) (xy 184.15 34.29)
+			(xy 149.86 20.32) (xy 157.48 20.32)
 		)
 		(stroke
@@
 	(wire
 		(pts
-			(xy 138.43 157.48) (xy 138.43 160.02)
+			(xy 181.61 34.29) (xy 184.15 34.29)
 		)
 		(stroke
@@
 	(wire
 		(pts
-			(xy 212.09 149.86) (xy 212.09 151.13)
+			(xy 138.43 157.48) (xy 138.43 160.02)
 		)
 		(stroke
@@
 	(wire
 		(pts
-			(xy 223.52 100.33) (xy 201.93 100.33)
+			(xy 212.09 149.86) (xy 212.09 151.13)
 		)
 		(stroke
@@
 	(wire
 		(pts
-			(xy 223.52 95.25) (xy 201.93 95.25)
-		)
-		(stroke
-			(width 0)
-			(type default)
-		)
-	)
-	(wire
-		(pts
 			(xy 124.46 59.69) (xy 124.46 52.07)
 		)
@@
 	)
 	(label "DBG_LED0"
-		(at 223.52 95.25 180)
+		(at 238.76 95.25 180)
 		(effects
 			(font
@@
 	)
 	(label "DBG_LED2"
-		(at 223.52 100.33 180)
+		(at 238.76 100.33 180)
 		(effects
 			(font
@@
 	)
 	(label "DBG_LED1"
-		(at 223.52 97.79 180)
+		(at 238.76 97.79 180)
 		(effects
 			(font
@@
 		)
 	)
+	(hierarchical_label "PC7{slash}I2C4_SDA"
+		(shape bidirectional)
+		(at 50.8 166.37 0)
+		(effects
+			(font
+				(size 1.27 1.27)
+			)
+			(justify left)
+		)
+	)
 	(hierarchical_label "PC6{slash}I2C4_SCL"
 		(shape output)
@@
 		)
 	)
-	(hierarchical_label "PC9{slash}I2C3_SDA"
-		(shape bidirectional)
-		(at 50.8 166.37 0)
-		(effects
-			(font
-				(size 1.27 1.27)
-			)
-			(justify left)
-		)
-	)
 	(hierarchical_label "PA8{slash}GPIO"
 		(shape bidirectional)
@@
 		)
 	)
-	(hierarchical_label "PB2{slash}GPIO"
-		(shape bidirectional)
+	(hierarchical_label "PB2{slash}RS485FC"
+		(shape output)
 		(at 201.93 92.71 0)
 		(effects
@@
 		)
 	)
-	(hierarchical_label "PB12{slash}RS485_FC"
+	(hierarchical_label "PC6{slash}I2C4_SCL"
 		(shape output)
+		(at 50.8 168.91 0)
+		(effects
+			(font
+				(size 1.27 1.27)
+			)
+			(justify left)
+		)
+	)
+	(hierarchical_label "PB12{slash}ADC41_IN3_11"
+		(shape input)
 		(at 201.93 118.11 0)
 		(effects
@@
 		)
 	)
+	(hierarchical_label "PC12{slash}GPIO"
+		(shape bidirectional)
+		(at 166.37 97.79 180)
+		(effects
+			(font
+				(size 1.27 1.27)
+			)
+			(justify right)
+		)
+	)
 	(hierarchical_label "PA3{slash}UART2_RX"
 		(shape input)
@@
 		)
 	)
-	(hierarchical_label "PC3{slash}ADC12_IN9"
+	(hierarchical_label "PC3{slash}GPIO"
 		(shape bidirectional)
 		(at 166.37 74.93 180)
@@
 		(effects
 			(font
-				(size 1.27 1.27)
-			)
-			(justify left)
-		)
-	)
-	(hierarchical_label "PC8{slash}I2C3_SCL"
-		(shape output)
-		(at 50.8 168.91 0)
-		(effects
-			(font
