File: uMule_board/uMule_board.kicad_pcb (KiCad board)
At the start: 2 copper layers, 140 x 140 mm, 154 parts, among them J1 12V IN, J10 Conn_01x04, J11 Conn_01x04, J12 Conn_01x04, J13 Conn_01x04, J2 Dynamixel, J3 Li-Dar_UART, J4 ESP32_UART, J5 Conn_ST_STDC14, J6 I2C, J7 SPI_IMU, J8 Conn_02x04_Odd_Even, J9 Conn_02x04_Odd_Even, P1 BPV10NF, P2 BPV10NF, P3 BPV10NF, P4 BPV10NF, P5 BPV10NF, P6 BPV10NF, P7 BPV10NF, P8 BPV10NF, Q1 AON6407, Q2 S9015, SW1 DBG_BUTT, SW2 RST, U1 TPS62933, U10 OPA397DBVR, U11 OPA397DBVR, U12 OPA397DBVR, U13 OPA397DBVR, U14 OPA397DBVR, U15 OPA397DBVR, U16 SP3485CN, U17 STM32G474RETx, U2 TLV761, U3 LM431BMC3, U4 INA219AxD, U5 TPS62933, U7 FM24C64B, U8 OPA397DBVR, U9 OPA397DBVR, Y1 8MHz

Commit message: All elements connected. Now making more vias and corrections
Parts:
- moved C38 36.7 mm to (168.7, 89.2)
- moved U7 36.6 mm to (169.7, 93.7)
- moved J7 18.4 mm to (153.8, 125.5), turned to 0 degrees
- moved D10 18.2 mm to (124.2, 95.5)
- moved D8 18.2 mm to (124.2, 99.1)
- moved D9 18.2 mm to (124.2, 97.3)
- moved R24 18.2 mm to (127.5, 99.1)
- moved R25 18.2 mm to (127.5, 97.3)
- moved R26 18.2 mm to (127.5, 95.5)
- moved C50 15.8 mm to (179.3, 127.3)
- moved J2 15.8 mm to (171.3, 138.4)
- moved D11 15.8 mm to (175.0, 132.3)
- moved R37 15.8 mm to (175.0, 129.5)
- moved U16 15.8 mm to (175.0, 124.7)
- moved J6 15.6 mm to (156.3, 145.8)
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Connections:
- J10 pad 1: unconnected-(J10-Pin_1-Pad1) -> /GPIO/GPIO_8
- J10 pad 2: /GPIO/GPIO_3 -> /GPIO/GPIO_9
- J10 pad 3: /GPIO/GPIO_4 -> /GPIO/GPIO_10
- J10 pad 4: /GPIO/GPIO_5 -> /GPIO/GPIO_13
- J11 pad 1: /GPIO/GPIO_6 -> /GPIO/GPIO_14
- J11 pad 2: unconnected-(J11-Pin_2-Pad2) -> /GPIO/GPIO_11
- J11 pad 3: unconnected-(J11-Pin_3-Pad3) -> /GPIO/GPIO_0
- J11 pad 4: /GPIO/GPIO_7 -> /GPIO/GPIO_1
- J12 pad 1: /GPIO/GPIO_8 -> /GPIO/GPIO_12
- J12 pad 2: /GPIO/GPIO_9 -> /GPIO/GPIO_15
- J12 pad 3: /GPIO/GPIO_10 -> /GPIO/GPIO_7
- J12 pad 4: /GPIO/GPIO_11 -> /GPIO/GPIO_6
- J13 pad 1: /GPIO/GPIO_12 -> /GPIO/GPIO_2
- J13 pad 2: /GPIO/GPIO_13 -> /GPIO/GPIO_3
- J13 pad 3: /GPIO/GPIO_1 -> /GPIO/GPIO_4
- J13 pad 4: /GPIO/GPIO_2 -> /GPIO/GPIO_5
- R20 pad 2: /MCU/PC8/I2C3_SCL -> /Communication/I2C_SCL
- R21 pad 2: /MCU/PC9/I2C3_SDA -> /Communication/I2C_SDA
- R38 pad 2: /Communication/I2C_SDA -> /MCU/PC7/I2C4_SDA
- R39 pad 2: /Communication/I2C_SCL -> /MCU/PC6/I2C4_SCL
- U17 pad 11: /Photodiodes/V_{REF} -> /GPIO/GPIO_11
- U17 pad 12: /GPIO_1 -> /GPIO/GPIO_0
- U17 pad 13: /GPIO_2 -> /GPIO/GPIO_1
- U17 pad 26: /GPIO_5 -> /Communication/RS485_FC
- U17 pad 3: /GPIO_14 -> /GPIO/GPIO_13
- U17 pad 34: /Communication/RS485_FC -> /Photodiodes/PHO_2
- U17 pad 35: /Photodiodes/PHO_2 -> /Photodiodes/V_{REF}
- U17 pad 38: /Communication/I2C_SCL -> /MCU/PC6/I2C4_SCL
- U17 pad 39: /Communication/I2C_SDA -> /MCU/PC7/I2C4_SDA
- U17 pad 4: /GPIO_15 -> /GPIO/GPIO_14
- U17 pad 40: /MCU/PC8/I2C3_SCL -> /Communication/I2C_SCL
- U17 pad 41: /MCU/PC9/I2C3_SDA -> /Communication/I2C_SDA
- U17 pad 42: /GPIO_3 -> /GPIO/GPIO_2
- U17 pad 43: /GPIO_4 -> /GPIO/GPIO_3
- U17 pad 44: /GPIO_7 -> /GPIO/GPIO_4
- U17 pad 45: /GPIO_8 -> /GPIO/GPIO_5
- U17 pad 46: /GPIO_9 -> /GPIO/GPIO_6
- U17 pad 51: /GPIO_10 -> /GPIO/GPIO_7
- U17 pad 54: unconnected-(U17-PC12-Pad54) -> /GPIO/GPIO_12
- U17 pad 55: /GPIO_11 -> /GPIO/GPIO_15
- U17 pad 59: /GPIO_12 -> /GPIO/GPIO_8
- U17 pad 60: /GPIO_13 -> /GPIO/GPIO_9
- U17 pad 62: /GPIO_6 -> /GPIO/GPIO_10
- U4 pad 3: /MCU/PC9/I2C3_SDA -> /MCU/PC7/I2C4_SDA
- U4 pad 4: /MCU/PC8/I2C3_SCL -> /MCU/PC6/I2C4_SCL
- U7 pad 5: /MCU/PC9/I2C3_SDA -> /MCU/PC7/I2C4_SDA
- U7 pad 6: /MCU/PC8/I2C3_SCL -> /MCU/PC6/I2C4_SCL
Routing:
- net +3V3: track 330.6 -> 441.6 mm, vias 9 -> 13
- net /Photodiodes/PHO_2: track 0.00 -> 76.7 mm
- net /Photodiodes/PHO_4: track 5.75 -> 79.6 mm, vias 0 -> 2
- net /Photodiodes/PHO_5: track 5.75 -> 79.6 mm, vias 0 -> 2
- net /Photodiodes/PHO_6: track 5.75 -> 79.6 mm, vias 0 -> 2
- net /Photodiodes/PHO_7: track 5.75 -> 79.6 mm, vias 0 -> 2
- net /Photodiodes/PHO_3: track 5.75 -> 79.5 mm, vias 0 -> 2
- net /Photodiodes/PHO_0: track 0.00 -> 73.7 mm, vias 0 -> 2
- net /Photodiodes/PHO_1: track 5.75 -> 79.3 mm, vias 0 -> 2
- net /Communication/I2C_SDA: track 0.00 -> 72.3 mm, vias 0 -> 1
- net /Communication/I2C_SCL: track 0.00 -> 69.9 mm, vias 0 -> 1
- net /GPIO/GPIO_9: track 0.00 -> 55.9 mm, vias 0 -> 2
- net /GPIO/GPIO_8: track 0.00 -> 55.1 mm, vias 0 -> 2
- net /GPIO/GPIO_10: track 0.00 -> 55.0 mm, vias 0 -> 2
- net /GPIO/GPIO_6: track 0.00 -> 50.5 mm, vias 0 -> 2
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
Commit message: Board finished, ready to order
Routing:
- net /Photodiodes/PHO_0: track 73.7 -> 79.5 mm
- net /Photodiodes/PHO_2: track 76.7 -> 82.5 mm
- net GND: vias 431 -> 3070
- net /Power/+5V: vias 3 -> 2
Other:
- board text added: "A"
- board text added: "C"
- board text added: "P10"
- board text added: "P11"
- board text added: "P12"
- board text added: "PA0"
- board text added: "PA1"
- board text added: "PA8"
- board text added: "PA9"
- board text added: "PB6"
- board text added: "PB7"
- board text added: "PC3"
- board text added: "PD2"
- board text removed: "NCX"
- board text removed: "P13"
- board text removed: "PB1"
- board text removed: "PB2"
- board text removed: "PB3"
- board text removed: "PB4"
- board text removed: "PB5"
- board text removed: "PC4"
- board text removed: "PC5"
- board text removed: "PC6"
- board text removed: "PC7"
- board text removed: "PC8"
- board text removed: "PC9"
