File: uMule_transmiter/sheets/led_controller.kicad_sch (KiCad schematic)
At the start: 17 parts, among them J1 Screw_Terminal_01x02, J2 Conn_01x01_Socket, U1 TPS61042

Commit message: JLC Ready, now waiting for shipment
Parts:
- U1: footprint Package_SON:VSON-8-1EP_3x3mm_P0.65mm_EP1.65x2.4mm -> Package_SON:Texas_S-PVSON-N8
Changed lines of the file:
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@@
 			)
 		)
-		(property "Footprint" "Package_SON:VSON-8-1EP_3x3mm_P0.65mm_EP1.65x2.4mm"
+		(property "Footprint" "Package_SON:Texas_S-PVSON-N8"
 			(at 66.04 62.23 0)
 			(effects
